File: kicad/rosalyn-sat.kicad_pcb (KiCad board)
At the start: 4 copper layers, 21 x 15 mm, 18 parts, among them J2 Serial, U1 STM32F030F4Px, U2 E22-EBYTE, U3 XC6206P330MR

Commit message: Tage (#2)
* rosalyn-sat_v1.0

* added nvdata driver

* removed kicad bak files

* removed stm32__ folder
Parts:
- U1: value STM32F030F4Px -> STM32F070F6Px
Connections:
- net e22_busy renamed radio_busy
- net e22_dio1 renamed radio_dio1
- net e22_dio2 renamed radio_dio2
- net e22_nrst renamed radio_nrst
- net e22_nss renamed radio_nss
- net e22_rxen renamed radio_rxen
- net e22_txen renamed radio_txen
